Commit message: Generate the F1TENTH meshes the URDF references, and test that they exist
The URDF referenced 21 meshes while 4 were on disk. Nothing failed:
robot_state_publisher never loads geometry, so the package's structural tests
and every launch passed while RViz would have drawn a vehicle with no
suspension, hubs, motors, compute module, battery or camera.

Runs the committed generator to produce the 18 missing meshes, and adds a
tier-1 case that resolves every mesh:// reference in the URDF against the
package -- the cheapest possible guard against a class of defect that is
invisible to every other test here.

Co-Authored-By: Claude Opus 5 <noreply@anthropic.com>

File: ros_ws/src/racing_vehicle_description/urdf/f1tenth.urdf (robot description, URDF)
Before this commit: robot f1tenth, 9 links, 8 joints
Links:
- removed link chassis
- added link battery_pack; visual mesh filename=package://racing_vehicle_description/meshes/battery_pack.stl
- added link camera; visual mesh filename=package://racing_vehicle_description/meshes/camera_box.stl
- added link front_hub_left; visual mesh filename=package://racing_vehicle_description/meshes/front_hub_left.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
- added link front_hub_right; visual mesh filename=package://racing_vehicle_description/meshes/front_hub_right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
- added link front_shock_left; visual mesh filename=package://racing_vehicle_description/meshes/front_shock_lef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
- added link front_shock_right; visual mesh filename=package://racing_vehicle_description/meshes/front_shock_rig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
- added link front_suspension_left; visual mesh filename=package://racing_vehicle_description/meshes/front_susp_left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
- added link front_suspension_right; visual mesh filename=package://racing_vehicle_description/meshes/front_susp_righ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
- added link jetson_board; visual mesh filename=package://racing_vehicle_description/meshes/jetson_board.stl
- added link motor_left; visual mesh filename=package://racing_vehicle_description/meshes/motor_left.stl
- added link motor_right; visual mesh filename=package://racing_vehicle_description/meshes/motor_right.stl
- added link rear_hub_left; visual mesh filename=package://racing_vehicle_description/meshes/rear_hub_left.s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
- added link rear_hub_right; visual mesh filename=package://racing_vehicle_description/meshes/rear_hub_right.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
- added link rear_shock_left; visual mesh filename=package://racing_vehicle_description/meshes/rear_shock_left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
- added link rear_shock_right; visual mesh filename=package://racing_vehicle_description/meshes/rear_shock_righ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
- added link rear_suspension_left; visual mesh filename=package://racing_vehicle_description/meshes/rear_susp_left.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
- added link rear_suspension_right; visual mesh filename=package://racing_vehicle_description/meshes/rear_susp_right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
- link base_link: geometry visual mesh filename=package://racing_vehicle_description/meshes/chassis.stl
- link laser: geometry visual mesh filename=package://racing_vehicle_description/meshes/hokuyo.stl scale=0.12 0.12 0.12
- link left_steering_hinge: geometry 
- link right_steering_hinge: geometry 
Joints:
- removed joint base_link_to_chassis
- removed joint chassis_to_left_rear_wheel
- removed joint chassis_to_left_steering_hinge
- removed joint chassis_to_right_rear_wheel
- removed joint chassis_to_right_steering_hinge
- added joint base_link_to_battery_pack: type fixed, parent base_link, child battery_pack
- added joint base_link_to_camera: type fixed, parent base_link, child camera
- added joint base_link_to_front_hub_left: type fixed, parent base_link, child front_hub_left
- added joint base_link_to_front_hub_right: type fixed, parent base_link, child front_hub_right
- added joint base_link_to_front_shock_left: type fixed, parent base_link, child front_shock_left
- added joint base_link_to_front_shock_right: type fixed, parent base_link, child front_shock_right
- added joint base_link_to_front_suspension_left: type fixed, parent base_link, child front_suspension_left
- added joint base_link_to_front_suspension_right: type fixed, parent base_link, child front_suspension_right
- added joint base_link_to_jetson_board: type fixed, parent base_link, child jetson_board
- added joint base_link_to_left_rear_wheel: type fixed, parent base_link, child left_rear_wheel, origin xyz=-0.0508 0.12065 0.0508 rpy=1.5708 0 0
- added joint base_link_to_left_steering_hinge: type fixed, parent base_link, child left_steering_hinge, origin xyz=0.3810 0.12065 0.0508 rpy=0 0 0
- added joint base_link_to_motor_left: type fixed, parent base_link, child motor_left
- added joint base_link_to_motor_right: type fixed, parent base_link, child motor_right
- added joint base_link_to_rear_hub_left: type fixed, parent base_link, child rear_hub_left
- added joint base_link_to_rear_hub_right: type fixed, parent base_link, child rear_hub_right
- added joint base_link_to_rear_shock_left: type fixed, parent base_link, child rear_shock_left
- added joint base_link_to_rear_shock_right: type fixed, parent base_link, child rear_shock_right
- added joint base_link_to_rear_suspension_left: type fixed, parent base_link, child rear_suspension_left
- added joint base_link_to_rear_suspension_right: type fixed, parent base_link, child rear_suspension_right
- added joint base_link_to_right_rear_wheel: type fixed, parent base_link, child right_rear_wheel, origin xyz=-0.0508 -0.12065 0.0508 rpy=1.5708 0 0
- added joint base_link_to_right_steering_hinge: type fixed, parent base_link, child right_steering_hinge, origin xyz=0.3810 -0.12065 0.0508 rpy=0 0 0
- joint base_link_to_laser: origin xyz=0.125 0.0 0.205 rpy=0 0 0 -> xyz=0.275 0.0 0.105 rpy=0 0 0
