Commit message: Replace placeholder URDF geometry with real F1TENTH meshes and fix RViz scan QoS mismatch

File: ros_ws/src/racing_vehicle_description/urdf/f1tenth.urdf (robot description, URDF)
Before this commit: robot f1tenth, 2 links, 1 joints
Links:
- added link chassis; visual mesh filename=package://racing_vehicle_description/meshes/chassis.stl scale=0.000990 0.0009375 0.0009375
- added link left_front_wheel; visual mesh filename=package://racing_vehicle_description/meshes/left_wheel.stl
- added link left_rear_wheel; visual mesh filename=package://racing_vehicle_description/meshes/left_wheel.stl
- added link left_steering_hinge; visual mesh filename=package://racing_vehicle_description/meshes/hinge.stl
- added link right_front_wheel; visual mesh filename=package://racing_vehicle_description/meshes/right_wheel.stl
- added link right_rear_wheel; visual mesh filename=package://racing_vehicle_description/meshes/right_wheel.stl
- added link right_steering_hinge; visual mesh filename=package://racing_vehicle_description/meshes/hinge.stl
- link base_link: geometry 
- link laser: geometry visual mesh filename=package://racing_vehicle_description/meshes/hokuyo.stl
Joints:
- added joint base_link_to_chassis: type fixed, parent base_link, child chassis, origin xyz=0 0 0.05 rpy=0 0 0
- added joint chassis_to_left_rear_wheel: type fixed, parent chassis, child left_rear_wheel, origin xyz=0 0.1 0 rpy=1.5708 0 0
- added joint chassis_to_left_steering_hinge: type fixed, parent chassis, child left_steering_hinge, origin xyz=0.325 0.1 0 rpy=0 1.5708 0
- added joint chassis_to_right_rear_wheel: type fixed, parent chassis, child right_rear_wheel, origin xyz=0 -0.1 0 rpy=1.5708 0 0
- added joint chassis_to_right_steering_hinge: type fixed, parent chassis, child right_steering_hinge, origin xyz=0.325 -0.1 0 rpy=0 1.5708 0
- added joint left_steering_hinge_to_left_front_wheel: type fixed, parent left_steering_hinge, child left_front_wheel, origin xyz=0 0 0 rpy=1.5708 0 0
- added joint right_steering_hinge_to_right_front_wheel: type fixed, parent right_steering_hinge, child right_front_wheel, origin xyz=0 0 0 rpy=1.5708 0 0
- joint base_link_to_laser: origin xyz=0.20 0.0 0.12 rpy=0 0 0 -> xyz=0.125 0.0 0.205 rpy=0 0 0

Commit message: This commit moves the URDF's wheel axles to x = 0 and 0.33 so they sit 0.33 m apart as the vehicle file's wheelbase says (they were 0.4318 m apart), rescales the wheels, and regenerates the meshes from the updated generators.
Refs #12

File: ros_ws/src/racing_vehicle_description/urdf/f1tenth.urdf (robot description, URDF)
Before this commit: robot f1tenth, 25 links, 24 joints
Links:
- link laser: geometry visual mesh filename=package://racing_vehicle_description/meshes/hokuyo.stl scale=1 1 1
- link left_front_wheel: geometry visual mesh filename=package://racing_vehicle_description/meshes/left_wheel.stl scale=1.16 1.16 1
- link left_rear_wheel: geometry visual mesh filename=package://racing_vehicle_description/meshes/left_wheel.stl scale=1.16 1.16 1
- link right_front_wheel: geometry visual mesh filename=package://racing_vehicle_description/meshes/right_wheel.stl scale=1.16 1.16 1
- link right_rear_wheel: geometry visual mesh filename=package://racing_vehicle_description/meshes/right_wheel.stl scale=1.16 1.16 1
Joints:
- joint base_link_to_left_rear_wheel: origin xyz=-0.0508 0.12065 0.0508 rpy=1.5708 0 0 -> xyz=0 0.118 0.058 rpy=1.5708 0 0
- joint base_link_to_left_steering_hinge: origin xyz=0.3810 0.12065 0.0508 rpy=0 0 0 -> xyz=0.33 0.118 0.058 rpy=0 0 0
- joint base_link_to_right_rear_wheel: origin xyz=-0.0508 -0.12065 0.0508 rpy=1.5708 0 0 -> xyz=0 -0.118 0.058 rpy=1.5708 0 0
- joint base_link_to_right_steering_hinge: origin xyz=0.3810 -0.12065 0.0508 rpy=0 0 0 -> xyz=0.33 -0.118 0.058 rpy=0 0 0

Commit message: This commit adds the cog_link frame to the URDF at the gym's (lr, 0, h), pinned to Param by SIMJAX-1150. Refs #12

File: ros_ws/src/racing_vehicle_description/urdf/f1tenth.urdf (robot description, URDF)
Before this commit: robot f1tenth, 25 links, 24 joints
Links:
- added link cog_link
Joints:
- added joint base_link_to_cog_link: type fixed, parent base_link, child cog_link, origin xyz=0.17145 0.0 0.074 rpy=0 0 0

Commit message: This commit roots the URDF at the centre of gravity and hangs the drawing off a new rear_axle child at (-lr, 0, -h), with SIMJAX-1140 and DESC-1020. Refs #12

File: ros_ws/src/racing_vehicle_description/urdf/f1tenth.urdf (robot description, URDF)
Before this commit: robot f1tenth, 25 links, 24 joints
Links:
- added link rear_axle; visual mesh filename=package://racing_vehicle_description/meshes/chassis.stl
- link base_link: geometry 
Joints:
- removed joint base_link_to_battery_pack
- removed joint base_link_to_camera
- removed joint base_link_to_front_hub_left
- removed joint base_link_to_front_hub_right
- removed joint base_link_to_front_shock_left
- removed joint base_link_to_front_shock_right
- removed joint base_link_to_front_suspension_left
- removed joint base_link_to_front_suspension_right
- removed joint base_link_to_jetson_board
- removed joint base_link_to_left_rear_wheel
- removed joint base_link_to_left_steering_hinge
- removed joint base_link_to_motor_left
- removed joint base_link_to_motor_right
- removed joint base_link_to_rear_hub_left
- removed joint base_link_to_rear_hub_right
- removed joint base_link_to_rear_shock_left
- removed joint base_link_to_rear_shock_right
- removed joint base_link_to_rear_suspension_left
- removed joint base_link_to_rear_suspension_right
- removed joint base_link_to_right_rear_wheel
- removed joint base_link_to_right_steering_hinge
- added joint base_link_to_rear_axle: type fixed, parent base_link, child rear_axle, origin xyz=-0.17145 0 -0.074 rpy=0 0 0
- added joint rear_axle_to_battery_pack: type fixed, parent rear_axle, child battery_pack
- added joint rear_axle_to_camera: type fixed, parent rear_axle, child camera
- added joint rear_axle_to_front_hub_left: type fixed, parent rear_axle, child front_hub_left
- added joint rear_axle_to_front_hub_right: type fixed, parent rear_axle, child front_hub_right
- added joint rear_axle_to_front_shock_left: type fixed, parent rear_axle, child front_shock_left
- added joint rear_axle_to_front_shock_right: type fixed, parent rear_axle, child front_shock_right
- added joint rear_axle_to_front_suspension_left: type fixed, parent rear_axle, child front_suspension_left
- added joint rear_axle_to_front_suspension_right: type fixed, parent rear_axle, child front_suspension_right
- added joint rear_axle_to_jetson_board: type fixed, parent rear_axle, child jetson_board
- added joint rear_axle_to_left_rear_wheel: type fixed, parent rear_axle, child left_rear_wheel, origin xyz=0 0.118 0.058 rpy=1.5708 0 0
- added joint rear_axle_to_left_steering_hinge: type fixed, parent rear_axle, child left_steering_hinge, origin xyz=0.33 0.118 0.058 rpy=0 0 0
- added joint rear_axle_to_motor_left: type fixed, parent rear_axle, child motor_left
- added joint rear_axle_to_motor_right: type fixed, parent rear_axle, child motor_right
- added joint rear_axle_to_rear_hub_left: type fixed, parent rear_axle, child rear_hub_left
- added joint rear_axle_to_rear_hub_right: type fixed, parent rear_axle, child rear_hub_right
- added joint rear_axle_to_rear_shock_left: type fixed, parent rear_axle, child rear_shock_left
- added joint rear_axle_to_rear_shock_right: type fixed, parent rear_axle, child rear_shock_right
- added joint rear_axle_to_rear_suspension_left: type fixed, parent rear_axle, child rear_suspension_left
- added joint rear_axle_to_rear_suspension_right: type fixed, parent rear_axle, child rear_suspension_right
- added joint rear_axle_to_right_rear_wheel: type fixed, parent rear_axle, child right_rear_wheel, origin xyz=0 -0.118 0.058 rpy=1.5708 0 0
- added joint rear_axle_to_right_steering_hinge: type fixed, parent rear_axle, child right_steering_hinge, origin xyz=0.33 -0.118 0.058 rpy=0 0 0
- joint base_link_to_laser: origin xyz=0.275 0.0 0.105 rpy=0 0 0 -> xyz=0.275 0.0 0.031 rpy=0 0 0

Commit message: This commit moves the laser joint to rear_axle_to_laser at 0.275 from the rear axle and casts /scan from laser_x - lr from the CoG, with BRINGUP-1050, SIMJAX-1090 and ADAPT-2120 expecting the true mount. Refs #12

File: ros_ws/src/racing_vehicle_description/urdf/f1tenth.urdf (robot description, URDF)
Before this commit: robot f1tenth, 26 links, 25 joints
Joints:
- removed joint base_link_to_laser
- added joint rear_axle_to_laser: type fixed, parent rear_axle, child laser, origin xyz=0.275 0.0 0.105 rpy=0 0 0

Commit message: This commit renames the lidar frame laser to lidar in the contract, the gym's /scan stamp and the URDF, and adds CHECK-2010/2020 to keep every copy of the name in step.

File: ros_ws/src/racing_vehicle_description/urdf/f1tenth.urdf (robot description, URDF)
Before this commit: robot f1tenth, 26 links, 25 joints
Links:
- removed link laser
- added link lidar; visual mesh filename=package://racing_vehicle_description/meshes/hokuyo.stl scale=1 1 1
Joints:
- removed joint rear_axle_to_laser
- added joint rear_axle_to_lidar: type fixed, parent rear_axle, child lidar, origin xyz=0.275 0.0 0.105 rpy=0 0 0
